File: board/wasca.sch (KiCad schematic (older format))
At the start: 70 parts, among them CN1 CARTRIDGE_EDGE_CONNECTOR, CON1 SD_Card, CON2 USB-MICRO-B, IC1 MT48LC32M16A2TG, U1 74ALVC164245, U2 74ALVC164245, U3 74ALVC164245, U4 74ALVC164245, U5 10M04SFE144C8G, U6 FT201XS

Commit message: Pre-route schematic. Kinda finished. Will change after route.
Parts:
- removed U?: AP1117E33, symbol AP1117E33
- added C13: 0.1uF, Capacitors_SMD:C_0603_HandSoldering, symbol C_Small
- added D1: D_Schottky_x2_KCom, Housings_SOT-23_SOT-143_TSOT-6:SOT-23_Handsoldering, symbol D_Schottky_x2_KCom
- added U5: LD1117S33CTR, SOT-223, symbol LD1117S33CTR
- gave numbers to parts that had none: 16
- renumbered C8 to C10, C9 to C11, C10 to C12, C11 to C14, C12 to C15, C13 to C16, C14 to C17, C15 to C18, C16 to C19, C1 to C2, C17 to C20, C18 to C21, C19 to C22, C20 to C23, C21 to C24, C22 to C26, C23 to C28, C24 to C29, C25 to C30, C26 to C32, C27 to C34, C28 to C35, C29 to C36, C30 to C37, C31 to C38, C2 to C4, C35 to C46, C37 to C48, C3 to C5, C4 to C6, C5 to C7, C6 to C8, C7 to C9, U5 to U6, U6 to U7
Connections:
- net labels added: USB_VBUS
- wire segments 628 -> 630
Other:
- note removed: "TODO:\n3.3V SOURCE\n\n"

Commit message: PCB preparement
Parts:
- U1, U2, U3, U4: footprint (none) -> Housings_SSOP:TSSOP-48_6.1x12.5mm_Pitch0.5mm
- U5: footprint SOT-223 -> SMD_Packages:SOT-223
- U6: footprint (none) -> Housings_QFP:TQFP-144_20x20mm_Pitch0.5mm
Changed lines of the file:
@@
 F 0 "U6" H 17350 8050 60  0000 C CNN
 F 1 "10M04SFE144C8G" H 15300 5150 60  0000 C CNN
-F 2 "" H 14950 4850 60  0000 C CNN
+F 2 "Housings_QFP:TQFP-144_20x20mm_Pitch0.5mm" H 14950 4850 60  0001 C CNN
 F 3 "" H 14950 4850 60  0000 C CNN
 	1    15300 4850
@@
 F 0 "CN1" H 4450 9050 60  0000 C CNN
 F 1 "CARTRIDGE_EDGE_CONNECTOR" H 4700 2000 60  0000 C CNN
-F 2 "" H 4700 5250 60  0000 C CNN
+F 2 "" H 4700 5250 60  0001 C CNN
 F 3 "" H 4700 5250 60  0000 C CNN
 	1    4700 5250
@@
 F 0 "U3" H 7950 6250 60  0000 L BNN
 F 1 "74ALVC164245" H 7950 6200 60  0000 L TNN
-F 2 "" H 8250 5000 60  0000 C CNN
+F 2 "Housings_SSOP:TSSOP-48_6.1x12.5mm_Pitch0.5mm" H 8250 5000 60  0001 C CNN
 F 3 "" H 8250 5000 60  0000 C CNN
 	1    8250 5350
@@
 F 0 "U1" H 4550 11000 60  0000 L BNN
 F 1 "74ALVC164245" H 4550 10950 60  0000 L TNN
-F 2 "" H 4850 9750 60  0000 C CNN
+F 2 "Housings_SSOP:TSSOP-48_6.1x12.5mm_Pitch0.5mm" H 4850 9750 60  0001 C CNN
 F 3 "" H 4850 9750 60  0000 C CNN
 	1    4850 10100
@@
 F 0 "U2" H 7950 2600 60  0000 L BNN
 F 1 "74ALVC164245" H 7950 2550 60  0000 L TNN
-F 2 "" H 8250 1350 60  0000 C CNN
+F 2 "Housings_SSOP:TSSOP-48_6.1x12.5mm_Pitch0.5mm" H 8250 1350 60  0001 C CNN
 F 3 "" H 8250 1350 60  0000 C CNN
 	1    8250 1700
@@
 F 0 "U4" H 8200 13200 60  0000 L BNN
 F 1 "74ALVC164245" H 8200 13150 60  0000 L TNN
-F 2 "" H 8500 11950 60  0000 C CNN
+F 2 "Housings_SSOP:TSSOP-48_6.1x12.5mm_Pitch0.5mm" H 8500 11950 60  0001 C CNN
 F 3 "" H 8500 11950 60  0000 C CNN
 	1    8500 12300
@@
 	1    0    0    -1
 $EndComp
-$Comp
-L USB-MICRO-B CON2
-U 1 1 5537B45B
-P 22000 3950
-F 0 "CON2" H 21700 4300 50  0000 C CNN
-F 1 "USB-MICRO-B" H 21850 3600 50  0000 C CNN
-F 2 "" H 22000 3850 50  0000 C CNN
-F 3 "" H 22000 3850 50  0000 C CNN
-	1    22000 3950
-	1    0    0    -1
-$EndComp
 Text Label 19400 1350 0    40   ~ 0
 +3_3V
@@
 F 0 "U5" H 15200 10200 40  0000 C CNN
 F 1 "LD1117S33CTR" H 15200 10150 40  0000 C CNN
-F 2 "SOT-223" H 15200 10050 40  0000 C CNN
+F 2 "SMD_Packages:SOT-223" H 15200 10050 40  0000 C CNN
 F 3 "" H 15200 9950 60  0000 C CNN
 	1    15200 9950
@@
 	14500 10000 14500 9900
 Connection ~ 14500 9900
+$Comp
+L USB-MICRO-B CON2
+U 1 1 5549505F
+P 22000 3950
+F 0 "CON2" H 21700 4300 50  0000 C CNN
+F 1 "USB-MICRO-B" H 21850 3600 50  0000 C CNN
+F 2 "" H 22000 3850 50  0000 C CNN
+F 3 "" H 22000 3850 50  0000 C CNN
+	1    22000 3950
+	1    0    0    -1
+$EndComp
 $EndSCHEMATC

Commit message: 
Parts:
- removed CON2: USB-MICRO-B, symbol USB-MICRO-B
- removed D1: D_Schottky_x2_KCom, Housings_SOT-23_SOT-143_TSOT-6:SOT-23_Handsoldering, symbol D_Schottky_x2_KCom
- added CON2: USB_OTG, symbol USB_OTG
- added D1: D_Schottky_x2_KCom_AAK, Housings_SOT-23_SOT-143_TSOT-6:SOT-23_Handsoldering, symbol D_Schottky_x2_KCom_AAK
Connections:
- wire segments 630 -> 625
Changed lines of the file:
@@
 LIBS:switches
 LIBS:maxim
-LIBS:wasca-cache
 EELAYER 25 0
 EELAYER END
@@
 L GND #PWR044
 U 1 1 5538C040
-P 22600 4200
-F 0 "#PWR044" H 22600 3950 50  0001 C CNN
-F 1 "GND" H 22600 4050 50  0001 C CNN
-F 2 "" H 22600 4200 60  0000 C CNN
-F 3 "" H 22600 4200 60  0000 C CNN
-	1    22600 4200
+P 21900 4350
+F 0 "#PWR044" H 21900 4100 50  0001 C CNN
+F 1 "GND" H 21900 4200 50  0001 C CNN
+F 2 "" H 21900 4350 60  0000 C CNN
+F 3 "" H 21900 4350 60  0000 C CNN
+	1    21900 4350
 	1    0    0    -1
 $EndComp
@@
 	21450 4150 21500 4150
 Wire Wire Line
-	22500 3750 22600 3750
-Wire Wire Line
-	22600 3750 22600 4200
-Wire Wire Line
-	22600 4150 22500 4150
-Wire Wire Line
-	22500 4050 22600 4050
-Connection ~ 22600 4050
-Wire Wire Line
-	22500 3850 22600 3850
-Connection ~ 22600 3850
-Connection ~ 22600 4150
-Wire Wire Line
 	20300 4150 20200 4150
 $Comp
@@
 USB_VBUS
 Wire Wire Line
-	13400 9700 13800 9700
+	13400 9700 14000 9700
 Text Label 13450 9700 0    40   ~ 0
 USB_VBUS
-$Comp
-L D_Schottky_x2_KCom D1
-U 1 1 554187D4
-P 14200 9700
-F 0 "D1" H 14350 9575 50  0000 C CNN
-F 1 "D_Schottky_x2_KCom" H 14200 9850 50  0000 C CNN
-F 2 "Housings_SOT-23_SOT-143_TSOT-6:SOT-23_Handsoldering" H 14150 10000 60  0000 C CNN
-F 3 "" H 14200 9700 60  0000 C CNN
-	1    14200 9700
-	1    0    0    -1
-$EndComp
 Wire Wire Line
 	14200 9900 14200 10000
@@
 Connection ~ 14500 9900
 $Comp
-L USB-MICRO-B CON2
-U 1 1 5549505F
-P 22000 3950
-F 0 "CON2" H 21700 4300 50  0000 C CNN
-F 1 "USB-MICRO-B" H 21850 3600 50  0000 C CNN
-F 2 "" H 22000 3850 50  0000 C CNN
-F 3 "" H 22000 3850 50  0000 C CNN
-	1    22000 3950
+L USB_OTG CON2
+U 1 1 5549E3D1
+P 21800 3950
+F 0 "CON2" H 22125 3825 50  0000 C CNN
+F 1 "USB_OTG" H 21800 4150 50  0000 C CNN
+F 2 "" V 21750 3850 60  0000 C CNN
+F 3 "" V 21750 3850 60  0000 C CNN
+	1    21800 3950
+	0    1    1    0
+$EndComp
+$Comp
+L D_Schottky_x2_KCom_AAK D1
+U 1 1 5549EFB4
+P 14300 9700
+F 0 "D1" H 14350 9600 50  0000 C CNN
+F 1 "D_Schottky_x2_KCom_AAK" H 14300 9800 50  0000 C CNN
+F 2 "Housings_SOT-23_SOT-143_TSOT-6:SOT-23_Handsoldering" H 14150 9950 60  0000 C CNN
+F 3 "" H 14300 9700 60  0000 C CNN
+	1    14300 9700
 	1    0    0    -1
 $EndComp

Commit message: 
Parts:
- CON1: footprint 10067847-001 -> Connect:SD_Card_Receptacle
- CON2: footprint (none) -> Connect:USB_Micro-B
- U7: footprint SSOP-16 -> Housings_SSOP:SSOP-16_3.9x4.9mm_Pitch0.635mm
Changed lines of the file:
@@
 F 0 "CON1" H 19650 2900 50  0000 C CNN
 F 1 "SD_Card" H 20900 1800 50  0000 C CNN
-F 2 "10067847-001" H 20500 2700 50  0000 C CNN
+F 2 "Connect:SD_Card_Receptacle" H 20500 2700 50  0000 C CNN
 F 3 "" H 20300 2350 60  0000 C CNN
 	1    20300 2350
@@
 F 0 "U7" H 18950 4550 50  0000 L CNN
 F 1 "FT201XS" H 19800 4550 50  0000 L CNN
-F 2 "SSOP-16" H 19500 3950 50  0000 C CNN
+F 2 "Housings_SSOP:SSOP-16_3.9x4.9mm_Pitch0.635mm" H 19500 3950 50  0000 C CNN
 F 3 "" H 19500 3950 50  0000 C CNN
 	1    19500 3950
@@
 F 0 "CON2" H 22125 3825 50  0000 C CNN
 F 1 "USB_OTG" H 21800 4150 50  0000 C CNN
-F 2 "" V 21750 3850 60  0000 C CNN
+F 2 "Connect:USB_Micro-B" V 21750 3850 60  0001 C CNN
 F 3 "" V 21750 3850 60  0000 C CNN
 	1    21800 3950

Commit message: PCB routing started
Parts:
- CN1: footprint (none) -> Wasca:CARTRIDGE_EDGE_CONNECTOR2
- IC1: footprint TSOPII-54 -> Wasca:TSOP_II_54
Changed lines of the file:
@@
 F 0 "IC1" H 19700 11500 40  0000 C CNN
 F 1 "MT48LC32M16A2TG" H 20950 9000 40  0000 C CNN
-F 2 "TSOPII-54" H 20300 10300 35  0000 C CIN
+F 2 "Wasca:TSOP_II_54" H 20300 10300 35  0000 C CIN
 F 3 "" H 20300 10050 60  0000 C CNN
 	1    20300 10300
@@
 F 0 "CN1" H 4450 9050 60  0000 C CNN
 F 1 "CARTRIDGE_EDGE_CONNECTOR" H 4700 2000 60  0000 C CNN
-F 2 "" H 4700 5250 60  0001 C CNN
+F 2 "Wasca:CARTRIDGE_EDGE_CONNECTOR2" H 4700 5250 60  0001 C CNN
 F 3 "" H 4700 5250 60  0000 C CNN
 	1    4700 5250

Commit message: Half-routed
Changed lines of the file:
@@
 Entry Wire Line
 	6600 7050 6700 6950
+Text Label 6900 6350 0    40   ~ 0
+ABUS_D7
+Text Label 6900 6450 0    40   ~ 0
+ABUS_D6
+Text Label 6900 6550 0    40   ~ 0
+ABUS_D5
+Text Label 6900 6650 0    40   ~ 0
+ABUS_D4
+Text Label 6900 6750 0    40   ~ 0
+ABUS_D15
+Text Label 6900 6850 0    40   ~ 0
+ABUS_D14
+Text Label 6900 6950 0    40   ~ 0
+ABUS_D13
 Text Label 6900 7050 0    40   ~ 0
-ABUS_D7
-Text Label 6900 6950 0    40   ~ 0
-ABUS_D6
-Text Label 6900 6850 0    40   ~ 0
-ABUS_D5
-Text Label 6900 6750 0    40   ~ 0
-ABUS_D4
-Text Label 6900 6650 0    40   ~ 0
-ABUS_D15
-Text Label 6900 6550 0    40   ~ 0
-ABUS_D14
-Text Label 6900 6450 0    40   ~ 0
-ABUS_D13
-Text Label 6900 6350 0    40   ~ 0
 ABUS_D12
 Entry Wire Line
@@
 	-1   0    0    -1
 $EndComp
-Text Label 6900 1900 0    40   ~ 0
+Text Label 6900 2700 0    40   ~ 0
 ABUS_FC1
-Text Label 6900 2000 0    40   ~ 0
+Text Label 6900 2300 0    40   ~ 0
 ABUS_TIM1
 Text Label 7150 13900 0    40   ~ 0
@@
 Text Label 7150 14000 0    40   ~ 0
 ABUS_IRQ
+Text Label 6900 3000 0    40   ~ 0
+ABUS_RD
+Text Label 6900 2900 0    40   ~ 0
+ABUS_CS1
+Text Label 6900 2800 0    40   ~ 0
+ABUS_WR1
+Text Label 6900 1900 0    40   ~ 0
+ABUS_FC0
+Text Label 6900 1800 0    40   ~ 0
+ABUS_TIM0
+Text Label 6900 1700 0    40   ~ 0
+ABUS_TIM2
 Text Label 6900 1600 0    40   ~ 0
-ABUS_RD
-Text Label 6900 1700 0    40   ~ 0
-ABUS_CS1
-Text Label 6900 1800 0    40   ~ 0
-ABUS_WR1
-Text Label 6900 2700 0    40   ~ 0
-ABUS_FC0
-Text Label 6900 2800 0    40   ~ 0
-ABUS_TIM0
-Text Label 6900 2900 0    40   ~ 0
-ABUS_TIM2
-Text Label 6900 3000 0    40   ~ 0
 ABUS_AS
+Text Label 6900 2200 0    40   ~ 0
+ABUS_CS0
 Text Label 6900 2100 0    40   ~ 0
-ABUS_CS0
-Text Label 6900 2200 0    40   ~ 0
 ABUS_CS2
-Text Label 6900 2300 0    40   ~ 0
+Text Label 6900 2000 0    40   ~ 0
 ABUS_WR0
 Text Label 7150 12200 0    40   ~ 0
 ABUS_A17
+Text Label 6900 3200 0    40   ~ 0
+ABUS_A23
 Text Label 6900 3300 0    40   ~ 0
-ABUS_A23
-Text Label 6900 3200 0    40   ~ 0
 ABUS_A21
+Text Label 6900 3400 0    40   ~ 0
+ABUS_A19
 Text Label 6900 3100 0    40   ~ 0
-ABUS_A19
-Text Label 6900 3400 0    40   ~ 0
 ABUS_A25
 Text Label 7150 12900 0    40   ~ 0
@@
 	6350 8250 6500 8250
 Wire Wire Line
+	6700 6350 7450 6350
+Wire Wire Line
+	6700 6450 7450 6450
+Wire Wire Line
+	6700 6550 7450 6550
+Wire Wire Line
+	6700 6650 7450 6650
+Wire Wire Line
+	6700 6750 7450 6750
+Wire Wire Line
+	6700 6850 7450 6850
+Wire Wire Line
+	6700 6950 7450 6950
+Wire Wire Line
 	6700 7050 7450 7050
-Wire Wire Line
-	6700 6950 7450 6950
-Wire Wire Line
-	6700 6850 7450 6850
-Wire Wire Line
-	6700 6750 7450 6750
-Wire Wire Line
-	6700 6650 7450 6650
-Wire Wire Line
-	6700 6550 7450 6550
-Wire Wire Line
-	6700 6450 7450 6450
-Wire Wire Line
-	6700 6350 7450 6350
 Wire Bus Line
 	6250 5150 6250 6050
@@
 	12300 3150 13050 3150
 Wire Wire Line
+	6700 2700 7450 2700
+Wire Wire Line
+	6700 2300 7450 2300
+Wire Wire Line
+	6950 13900 7700 13900
+Wire Wire Line
+	6950 14000 7700 14000
+Wire Wire Line
+	6700 3000 7450 3000
+Wire Wire Line
+	6700 2900 7450 2900
+Wire Wire Line
+	6700 2800 7450 2800
+Wire Wire Line
 	6700 1900 7450 1900
 Wire Wire Line
+	6700 1800 7450 1800
+Wire Wire Line
+	6700 1700 7450 1700
+Wire Wire Line
+	6700 1600 7450 1600
+Wire Wire Line
+	6700 2200 7450 2200
+Wire Wire Line
+	6700 2100 7450 2100
+Wire Wire Line
 	6700 2000 7450 2000
 Wire Wire Line
-	6950 13900 7700 13900
-Wire Wire Line
-	6950 14000 7700 14000
-Wire Wire Line
-	6700 1600 7450 1600
-Wire Wire Line
-	6700 1700 7450 1700
-Wire Wire Line
-	6700 1800 7450 1800
-Wire Wire Line
-	6700 2700 7450 2700
-Wire Wire Line
-	6700 2800 7450 2800
-Wire Wire Line
-	6700 2900 7450 2900
-Wire Wire Line
-	6700 3000 7450 3000
-Wire Wire Line
-	6700 2100 7450 2100
-Wire Wire Line
-	6700 2200 7450 2200
-Wire Wire Line
-	6700 2300 7450 2300
-Wire Wire Line
 	6950 12200 7700 12200
 Wire Wire Line
+	6700 3200 7450 3200
+Wire Wire Line
 	6700 3300 7450 3300
 Wire Wire Line
-	6700 3200 7450 3200
+	6700 3400 7450 3400
 Wire Wire Line
 	6700 3100 7450 3100
 Wire Wire Line
-	6700 3400 7450 3400
-Wire Wire Line
 	6950 12900 7700 12900

Commit message: Routed at last.
Parts:
- removed C17, C18, C19, C20, C21, C22, C29, C30, C49: 0.1uF, Capacitors_SMD:C_0603_HandSoldering, symbol C_Small
- removed D1: D_Schottky_x2_KCom_AAK, Housings_SOT-23_SOT-143_TSOT-6:SOT-23_Handsoldering, symbol D_Schottky_x2_KCom_AAK
- added CON3: Thermal_Quad, symbol Thermal_Quad
- added D1: D_Schottky_x2_KCom, Housings_SOT-23_SOT-143_TSOT-6:SOT-23_Handsoldering, symbol D_Schottky_x2_KCom
Connections:
- net labels added: USB_CBUS0, USB_CBUS1, USB_SCL, USB_SDA
- wire segments 625 -> 620
