File: board/wasca.sch (KiCad schematic (older format))
At the start: 64 parts, among them CN1 CARTRIDGE_EDGE_CONNECTOR, CON1 SD_Card, CON2 USB_OTG, CON3 Thermal_Quad, IC1 MT48LC32M16A2TG, U1 74ALVC164245, U2 74ALVC164245, U3 74ALVC164245, U4 74ALVC164245, U5 LD1117S33CTR, U6 10M04SFE144C8G, U7 FT201XS

Commit message: SCSP 22.57 MHz clock is used instead of 27..29 MHz MCLK2
Connections:
- net labels added: SCSPCLK, SCSPCLK_3V
- net labels removed: DOTCLK, DOTCLK_3V
- wire segments 620 -> 816

Commit message: Silkscreen cleanup
Parts:
- renumbered IC1 to U8
Connections:
- wire segments 816 -> 620

Commit message: Major board fixes
Parts:
- removed C45, C46, C48: 0.1uF, Capacitors_SMD:C_0603_HandSoldering, symbol C_Small
- removed CON3: Thermal_Quad, symbol Thermal_Quad
- removed D1: D_Schottky_x2_KCom, Housings_SOT-23_SOT-143_TSOT-6:SOT-23_Handsoldering, symbol D_Schottky_x2_KCom
- removed L1: L_Small, Resistors_SMD:R_0603_HandSoldering, symbol L_Small
- removed R8: 4.7K, Resistors_SMD:R_0603_HandSoldering, symbol R
- removed U6: 10M04SFE144C8G, Housings_QFP:TQFP-144_20x20mm_Pitch0.5mm, symbol 10M04SFE144C8G
- removed U7: FT201XS, Housings_SSOP:SSOP-16_3.9x4.9mm_Pitch0.635mm, symbol FT201XS
- removed U8: MT48LC32M16A2TG, Wasca:TSOP_II_54, symbol MT48LC32M16A2TG
- added A1: ANT, Wasca:PCB_IF_ANT_2.4G, symbol ANT
- added B1: 2450BM14E0003, Wasca:2450BM14E0003, symbol 2450BM14E0003
- added C10, C11: 47pF, Capacitors_SMD:C_0603_HandSoldering, symbol C_Small
- added C20, C21, C22, C23, C24, C25, C26, C27, C50, C51, C52, C53, C55: 0.1uF, Capacitors_SMD:C_0603_HandSoldering, symbol C_Small
- added C28: 10uF, Capacitors_SMD:C_1206_HandSoldering, symbol C_Small
- added C54: 47nF, Capacitors_SMD:C_0603_HandSoldering, symbol C_Small
- added C56: 2.2nF, Capacitors_SMD:C_0603_HandSoldering, symbol C_Small
- added CON3: AVR-JTAG-10, Pin_Headers:Pin_Header_Angled_2x05, symbol AVR-JTAG-10
- added CON4, CON5: AVR-ISP-6, Pin_Headers:Pin_Header_Angled_2x03, symbol AVR-ISP-6
- added D1: D_Schottky_x2_KCom_AAK, Housings_SOT-23_SOT-143_TSOT-6:SOT-23_Handsoldering, symbol D_Schottky_x2_KCom_AAK
- added JP1: JUMPER, Pin_Headers:Pin_Header_Straight_2x01, symbol JUMPER
- added R10, R11: 4.7K, Resistors_SMD:R_0603_HandSoldering, symbol R
- added R12, R13, R14: 50K, Resistors_SMD:R_0603_HandSoldering, symbol R
- added R15: 1K, Resistors_SMD:R_0603_HandSoldering, symbol R
- added R16, R17: 10K, Resistors_SMD:R_0603_HandSoldering, symbol R
- added R18: 12K, Resistors_SMD:R_0603_HandSoldering, symbol R
- added R5: DO NOT PLACE, Resistors_SMD:R_0603_HandSoldering, symbol R
- added U10: STM32F042C6T6, Housings_QFP:LQFP-48_7x7mm_Pitch0.5mm, symbol STM32F042C6T6
- added U11: 74ALVC164245, Housings_SSOP:TSSOP-48_6.1x12.5mm_Pitch0.5mm, symbol 74ALVC164245
- added U12: NRF51822, Wasca:QFN48_EXP, symbol NRF51822
- added U6: LD1117S25CTR, TO_SOT_Packages_SMD:SOT-223, symbol LD1117S25CTR
- added U7: DDR_SDRAM_MT46_x16, Wasca:TSOP66_JEDEC_DDR_SDRAM, symbol DDR_SDRAM_MT46_x16
- added U8: 10M04SFE144C8G, Wasca:TQFP144_ALTERA_HANDSOLDERING, symbol 10M04SFE144C8G
- added U9: SDRAM_MT48_x16, Wasca:TSOPII54_SDRAM_MT48, symbol SDRAM_MT48_x16
- added Y1: 16MHz, Crystals:Crystal_HC49-SD_SMD, symbol Crystal
- R1: renamed from R6; value 27 -> 33
- R2: renamed from R7; value 27 -> 33
- R9: value 4.7K -> 1K
- U5: footprint SMD_Packages:SOT-223 -> TO_SOT_Packages_SMD:SOT-223
- renumbered C8 to C12, C9 to C13, C25 to C14, C27 to C15, C31 to C16, C33 to C17, C43 to C18, C41 to C19, C11 to C29, C7 to C3, C14 to C30, C12 to C31, C15 to C32, C13 to C33, C16 to C34, C23 to C35, C24 to C36, C26 to C37, C28 to C38, C32 to C39, C3 to C4, C39 to C40, C34 to C41, C35 to C42, C40 to C43, C36 to C44, C42 to C45, C37 to C46, C38 to C47, C47 to C48, C50 to C49, C4 to C5, C10 to C6, C5 to C7, C6 to C8, C44 to C9, CON2 to CON1, CON1 to CON2, R5 to R3, R3 to R6, R2 to R7, R1 to R8, U4 to U2, U2 to U3, U3 to U4
Connections:
- net labels added: BLUE_CLK, BLUE_MISO, BLUE_MOSI, BLUE_SS, COMM_CLK, COMM_MISO, COMM_MOSI, COMM_SS, DDR_CLKN, DDR_DQSH, DDR_DQSL, IBCK, IBCK_3V, ILRCK, ILRCK_3V, ISD, ISD_3V, SSEL, SSEL_3V, VCC_SDRAM, WAIT_ENABLE
- net labels removed: ABUS_3V_AS, ABUS_3V_FC0, ABUS_3V_FC1, ABUS_3V_TIM0, ABUS_3V_TIM1, ABUS_3V_TIM2, ABUS_AS, ABUS_FC0, ABUS_FC1, ABUS_TIM0, ABUS_TIM1, ABUS_TIM2, USB_CBUS0, USB_CBUS1, USB_SCL, USB_SDA
- wire segments 620 -> 795

Commit message: Board 1.1 released
Parts:
- removed B1: 2450BM14E0003, Wasca:2450BM14E0003, symbol 2450BM14E0003
- removed C56: 2.2nF, Capacitors_SMD:C_0603_HandSoldering, symbol C_Small
- removed U12: NRF51822, Wasca:QFN48_EXP, symbol NRF51822
- added U12: CY8C4127LQI-BL473, Wasca:QFN56_EXP, symbol CY8C4127LQI-BL473
- added Y2: 32678Hz, Wasca:Crystal_5x3.2mm, symbol Crystal
- C26, C27: value 0.1uF -> 47pF
- C52, C53: value 0.1uF -> 1uF
- C54: value 47nF -> 0.1uF
- CON1: footprint Connect:USB_Micro-B -> Wasca:MicroUSB
- CON3: footprint Pin_Headers:Pin_Header_Angled_2x05 -> Wasca:Pinhead_2x5_SMD
- CON4, CON5: footprint Pin_Headers:Pin_Header_Angled_2x03 -> Wasca:Pinhead_2x3_SMD
- Y1: value 16MHz -> 24MHz; footprint Crystals:Crystal_HC49-SD_SMD -> Wasca:Crystal_5x3.2mm
Connections:
- wire segments 795 -> 784

Commit message: Board v1.2
Parts:
- removed A1: ANT, Wasca:PCB_IF_ANT_2.4G, symbol ANT
- removed C10, C11, C26, C27: 47pF, Capacitors_SMD:C_0603_HandSoldering, symbol C_Small
- removed C14, C28: 10uF, Capacitors_SMD:C_1206_HandSoldering, symbol C_Small
- removed C16, C19, C20, C21, C22, C23, C24, C25, C54, C55, C9: 0.1uF, Capacitors_SMD:C_0603_HandSoldering, symbol C_Small
- removed C18, C52, C53: 1uF, Capacitors_SMD:C_0603_HandSoldering, symbol C_Small
- removed CON1: USB_OTG, Wasca:MicroUSB, symbol USB_OTG
- removed CON2: SD_Card, Connect:SD_Card_Receptacle, symbol SD_Card
- removed CON4, CON5: AVR-ISP-6, Wasca:Pinhead_2x3_SMD, symbol AVR-ISP-6
- removed D1: D_Schottky_x2_KCom_AAK, Housings_SOT-23_SOT-143_TSOT-6:SOT-23_Handsoldering, symbol D_Schottky_x2_KCom_AAK
- removed JP1: JUMPER, Pin_Headers:Pin_Header_Straight_2x01, symbol JUMPER
- removed R1, R2: 33, Resistors_SMD:R_0603_HandSoldering, symbol R
- removed R10, R11: 4.7K, Resistors_SMD:R_0603_HandSoldering, symbol R
- removed R18: 12K, Resistors_SMD:R_0603_HandSoldering, symbol R
- removed R3, R4, R6, R8: 50K, Resistors_SMD:R_0603_HandSoldering, symbol R
- removed R5: DO NOT PLACE, Resistors_SMD:R_0603_HandSoldering, symbol R
- removed R9: 1K, Resistors_SMD:R_0603_HandSoldering, symbol R
- removed U10: STM32F042C6T6, Housings_QFP:LQFP-48_7x7mm_Pitch0.5mm, symbol STM32F042C6T6
- removed U12: CY8C4127LQI-BL473, Wasca:QFN56_EXP, symbol CY8C4127LQI-BL473
- removed U6: LD1117S25CTR, TO_SOT_Packages_SMD:SOT-223, symbol LD1117S25CTR
- removed U7: DDR_SDRAM_MT46_x16, Wasca:TSOP66_JEDEC_DDR_SDRAM, symbol DDR_SDRAM_MT46_x16
- removed Y1: 24MHz, Wasca:Crystal_5x3.2mm, symbol Crystal
- removed Y2: 32678Hz, Wasca:Crystal_5x3.2mm, symbol Crystal
- added C91: 4.7uF, Capacitors_SMD:C_0603_HandSoldering, symbol C_Small
- added LEDG1, LEDR1: LED, LEDs:LED-3MM, symbol LED
- added LEDR2: LED, LEDs:LED_0805, symbol LED
- added P84: CONN_01X02, Pin_Headers:Pin_Header_Straight_1x02, symbol CONN_01X02
- added R421, R422, R423: 470, Resistors_SMD:R_0603_HandSoldering, symbol R
- added R61, R62: 1K, Resistors_SMD:R_0603_HandSoldering, symbol R
- added R92: 51K, Resistors_SMD:R_0603_HandSoldering, symbol R
- added SD1: SD_CARD, wasca:sd_socket, symbol SD_CARD
- added X1, X61: CONN_02X02, Pin_Headers:Pin_Header_Straight_2x02, symbol CONN_02X02
- added X2, X3: CONN_02X05, Pin_Headers:Pin_Header_Straight_2x05, symbol CONN_02X05
- added X4: CONN_01X04, Pin_Headers:Pin_Header_Straight_1x04, symbol CONN_01X04
- C1: value 10uF -> 4.7uF
- C4: value 0.1uF -> 4.7uF
- CN1: footprint Wasca:CARTRIDGE_EDGE_CONNECTOR2 -> wasca:CARTRIDGE_EDGE_CONNECTOR2
- JTAG1: renamed from CON3; footprint Wasca:Pinhead_2x5_SMD -> wasca:JTAG_Header
- R12, R13, R14: value 50K -> 10K
- R91: renamed from R7; value 50K -> 51K
- U8: value 10M04SFE144C8G -> 10M08SCE144I7G; footprint Wasca:TQFP144_ALTERA_HANDSOLDERING -> wasca:TQFP144_ALTERA_HANDSOLDERING; symbol 10M04SFE144C8G -> 10M08SCE144I7G
- U9: footprint Wasca:TSOPII54_SDRAM_MT48 -> wasca:TSOPII54_SDRAM_MT48
- renumbered C17 to C16
Connections:
- net labels added: ABUS_FC0, ABUS_FC1, ABUS_TIM0, DDR_SPARE1, DDR_SPARE2, DDR_SPARE3, LEDG1, LEDR1, SD_CLK, SD_CS, SD_DIN, SD_DOUT, USB_CS, USB_RD, USB_SPARE1, USB_SPARE2
- net labels removed: BLUE_CLK, BLUE_MISO, BLUE_MOSI, BLUE_SS, COMM_CLK, COMM_MISO, COMM_MOSI, COMM_SS, DDR_CLKN, DDR_DQSH, DDR_DQSL, USB_VBUS
- wire segments 784 -> 713
- no-connect marks 0 -> 73
Other:
- note added: "--- Changelog ---\nV1.0 hitomi2500 :\n - Initial version with 10M04SFE, SDRAM, FT201XS\nV1.1 hitomi2500 :\n - Both DDR/SDRAM support\n - Added USB and bluetooth support\n - Sound I/O mapped to MAX10\nV1.2 cafe-alpha :\n - Changed PCB shape and ICs position in order to fit Action Replay case\n - Changed MAX10 chip from 10M04SFE to 10M08SCE\n - Changed SD card footprint to the one used in Gamer's C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"
- note added: "Connection with USB mezzanine board"
- note added: "External 5V power supply\n+ 3V3 power output/check"
- note added: "SDRAM : shares 3V3 with MAX10\nDDR : requires 2V5 power supply"
- note added: "Spare for DDR :\n - DDR_DQSH\n - DDR_DQSL\n - DDR_CLKN"
- note added: "Spare pull-up/down resistors"
- note added: "USB dev cart\n(EPM3064)"
