File: board/wasca.kicad_sch (KiCad schematic)
At the start: 62 parts, among them CN1 CARTRIDGE_EDGE_CONNECTOR, CN2 TFP09-2-12B, CN3 Conn_02x02_Odd_Even, CN4 SODIMM-200, U1 74ALVC164245, U10 SN74LVC1T45DBV, U11 SN74LVC1T45DBV, U12 SN74LVC1T45DBV, U13 ESP32_CAM_HALF, U2 74ALVC164245, U3 MT48LC16M16A2TG, U4 LD1117S33TR_SOT223, U5 74ALVC164245, U8 SN74LVC1T45DBV, U9 SN74LVC1T45DBV

Commit message: Test points
Parts:
- added TP1: TestPoint, wasca:TEST_PAD, symbol Connector:TestPoint
- added TP2: (no value), symbol Connector:TestPoint
- CN5: value (none) -> 693063020911; footprint (none) -> wasca:693063020911
Connections:
- net at CN4.150: now also TP2.1
- net at CN4.89: now also TP1.1
Changed lines of the file:
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@@
     (stroke (width 0) (type default) (color 0 0 0 0))
   )
+  (wire (pts (xy 604.52 118.11) (xy 645.16 118.11))
+    (stroke (width 0) (type default) (color 0 0 0 0))
+  )
   (wire (pts (xy 240.03 116.84) (xy 240.03 114.3))
     (stroke (width 0) (type default) (color 0 0 0 0))
@@
     (stroke (width 0) (type default) (color 0 0 0 0))
   )
+  (wire (pts (xy 680.72 194.31) (xy 713.74 194.31))
+    (stroke (width 0) (type default) (color 0 0 0 0))
+  )
   (wire (pts (xy 276.86 294.64) (xy 233.68 294.64))
     (stroke (width 0) (type default) (color 0 0 0 0))
@@
       (effects (font (size 1.27 1.27)) (justify left bottom))
     )
-    (property "Value" "" (id 1) (at 779.78 375.92 0)
+    (property "Value" "693063020911" (id 1) (at 779.78 375.92 0)
       (effects (font (size 1.27 1.27)) (justify left bottom))
     )
-    (property "Footprint" "" (id 2) (at 781.05 341.63 0)
+    (property "Footprint" "wasca:693063020911" (id 2) (at 781.05 341.63 0)
       (effects (font (size 1.27 1.27)) (justify left bottom) hide)
     )
@@
     (pin "WP")
   )
+  (symbol (lib_id "Connector:TestPoint") (at 604.52 118.11 0) (unit 1)
+    (in_bom yes) (on_board yes) (fields_autoplaced)
+    (property "Reference" "TP1" (id 0) (at 607.06 113.5379 0)
+      (effects (font (size 1.27 1.27)) (justify left))
+    )
+    (property "Value" "TestPoint" (id 1) (at 607.06 116.0779 0)
+      (effects (font (size 1.27 1.27)) (justify left))
+    )
+    (property "Footprint" "wasca:TEST_PAD" (id 2) (at 609.6 118.11 0)
+      (effects (font (size 1.27 1.27)) hide)
+    )
+    (property "Datasheet" "~" (id 3) (at 609.6 118.11 0)
+      (effects (font (size 1.27 1.27)) hide)
+    )
+    (pin "1")
+  )
   (symbol (lib_id "power:GND") (at 739.14 82.55 0) (unit 1)
     (in_bom yes) (on_board yes)
@@
     (pin "2")
   )
+  (symbol (lib_id "Connector:TestPoint") (at 713.74 194.31 0) (unit 1)
+    (in_bom yes) (on_board yes) (fields_autoplaced)
+    (property "Reference" "TP2" (id 0) (at 716.28 189.7379 0)
+      (effects (font (size 1.27 1.27)) (justify left))
+    )
+    (property "Value" "" (id 1) (at 716.28 192.2779 0)
+      (effects (font (size 1.27 1.27)) (justify left))
+    )
+    (property "Footprint" "" (id 2) (at 718.82 194.31 0)
+      (effects (font (size 1.27 1.27)) hide)
+    )
+    (property "Datasheet" "~" (id 3) (at 718.82 194.31 0)
+      (effects (font (size 1.27 1.27)) hide)
+    )
+    (pin "1")
+  )
   (sheet_instances
     (path "/" (page "1"))
@@
       (reference "SEGATA1") (unit 1) (value "LOGO") (footprint "wasca:Segata_Sanshiro")
     )
+    (path "/d276ace0-aa98-4013-94e5-a87cfcb3830a"
+      (reference "TP1") (unit 1) (value "TestPoint") (footprint "wasca:TEST_PAD")
+    )
+    (path "/f8083680-dc4d-419b-ad61-e71a2772eda6"
+      (reference "TP2") (unit 1) (value "TestPoint") (footprint "wasca:TEST_PAD")
+    )
     (path "/00000000-0000-0000-0000-00005536e7a3"
