File: board/wasca.kicad_sch (KiCad schematic)
At the start: 64 parts, among them CN1 CARTRIDGE_EDGE_CONNECTOR, CN2 TFP09-2-12B, CN3 Conn_02x02_Odd_Even, CN4 SODIMM-200, CN5 693063020911, CN6 Conn_01x02_Pin, U1 74ALVC164245, U10 SN74LVC1T45DBV, U11 SN74LVC1T45DBV, U12 SN74LVC1T45DBV, U13 ESP32_CAM_HALF, U2 74ALVC164245, U3 MT48LC16M16A2TG, U4 LD1117S33TR_SOT223, U5 74ALVC164245, U8 SN74LVC1T45DBV, U9 SN74LVC1T45DBV

Commit message: Adding FPGA+power supplies
Parts:
- added U14, U7: SY8008CAAC, wasca:SOT23-5_SY8008B_SGY, symbol sy8008:SY8008CAAC
- added U6: LFE5U-25F-6BG256I, wasca:caBGA256_LAT, symbol lfe5:LFE5U-25F-6BG256I
Connections:
- net GND: now also U6.A1 (GND), U6.A16 (GND), U6.D15 (GND), U6.D2 (GND), U6.F8 (GND), U6.F9 (GND), U6.G10 (GND), U6.G8 (GND), U6.H1 (GND), U6.H10 (GND), U6.H16 (GND), U6.H8 (GND), U6.H9 (GND), U6.J10 (GND), U6.J8 (GND), U6.J9 (GND), U6.K10 (GND), U6.K6 (GND), U6.K7 (GND), U6.K8 (GND), U6.K9 (GND), U6.N15 (GND), U6.N2 (GND), U6.T1 (GND), U6.T12 (GND), U6.T16 (GND), U6.T5 (GND)

Commit message: Board rerouting
Parts:
- removed C38, C52, C53: 0.1uF, Capacitor_SMD:C_0603_1608Metric_Pad1.08x0.95mm_HandSolder, symbol Device:C_Small
- removed CHAMFER_WARN1, CHAMFER_WARN2: CHAMFER_WARNING, wasca:CHAMFER_WARNING, symbol wasca:CHAMFER_WARNING
- removed CN3: Conn_02x02_Odd_Even, Connector_PinHeader_2.54mm:PinHeader_2x02_P2.54mm_Vertical, symbol Connector_Generic:Conn_02x02_Odd_Even
- removed CN4: SODIMM-200, wasca:Conn_TE-DDR2-SODIMM-0.6-200P-doublesided, symbol Connector:SODIMM-200
- removed CN6: Conn_01x02_Pin, Connector_PinHeader_2.54mm:PinHeader_1x02_P2.54mm_Vertical, symbol Connector:Conn_01x02_Pin
- removed U4: LD1117S33TR_SOT223, Package_TO_SOT_SMD:SOT-223-3_TabPin2, symbol Regulator_Linear:LD1117S33TR_SOT223
- added C10, C11, C12, C13, C14, C15, C16, C6, C7, C8, C9: 0.1uF, Capacitor_SMD:C_0402_1005Metric, symbol Device:C_Small
- added C18: 4.7uF, Capacitor_SMD:C_0603_1608Metric_Pad1.08x0.95mm_HandSolder, symbol Device:C_Small
- added C19, C20: 15pF, Capacitor_SMD:C_0603_1608Metric_Pad1.08x0.95mm_HandSolder, symbol Device:C_Small
- added C27, C28: 1uF, Capacitor_SMD:C_0603_1608Metric_Pad1.08x0.95mm_HandSolder, symbol Device:C_Small
- added C29, C31: 18pF, Capacitor_SMD:C_0603_1608Metric_Pad1.08x0.95mm_HandSolder, symbol Device:C_Small
- added C30, C32: 10uF, Capacitor_SMD:C_1206_3216Metric_Pad1.33x1.80mm_HandSolder, symbol Device:C_Small
- added C33, C34, C35, C36, C5, C56, C57, C58, C59, C60, C61, C62, C68: 0.1uF, Capacitor_SMD:C_0603_1608Metric_Pad1.08x0.95mm_HandSolder, symbol Device:C_Small
- added C66, C67: 22uF, Capacitor_SMD:C_0603_1608Metric_Pad1.08x0.95mm_HandSolder, symbol Device:C_Small
- added CN3: USB_C_Receptacle_USB2.0_16P, wasca:DX07S016JA1R1500, symbol Connector:USB_C_Receptacle_USB2.0_16P
- added D3: LED, LED_SMD:LED_0603_1608Metric, symbol Device:LED
- added L1, L2: 2.2uH, Inductor_SMD:L_1008_2520Metric, symbol Device:L
- added R12, R13: 5.1K, Resistor_SMD:R_0603_1608Metric_Pad0.98x0.95mm_HandSolder, symbol Device:R
- added R14, R18: 27, Resistor_SMD:R_0603_1608Metric_Pad0.98x0.95mm_HandSolder, symbol Device:R
- added R20, R30, R31: 1K, Resistor_SMD:R_0603_1608Metric_Pad0.98x0.95mm_HandSolder, symbol Device:R
- added R22, R25, R32, R39, R40: 0, Resistor_SMD:R_0603_1608Metric_Pad0.98x0.95mm_HandSolder, symbol Device:R
- added R23, R24, R33, R34, R35, R36, R37, R38: 10K, Resistor_SMD:R_0603_1608Metric_Pad0.98x0.95mm_HandSolder, symbol Device:R
- added R26: 680K, Resistor_SMD:R_0603_1608Metric_Pad0.98x0.95mm_HandSolder, symbol Device:R
- added R27: 150K, Resistor_SMD:R_0603_1608Metric_Pad0.98x0.95mm_HandSolder, symbol Device:R
- added R28: 200K, Resistor_SMD:R_0603_1608Metric_Pad0.98x0.95mm_HandSolder, symbol Device:R
- added R29: 240K, Resistor_SMD:R_0603_1608Metric_Pad0.98x0.95mm_HandSolder, symbol Device:R
- added R6: 4K7, Resistor_SMD:R_0603_1608Metric_Pad0.98x0.95mm_HandSolder, symbol Device:R
- added SW1: SW_Push, Button_Switch_SMD:SW_SPST_EVQP2_ShortPushTravel_H2.5mm, symbol Switch:SW_Push
- added SW2: SW_Push, symbol Switch:SW_Push
- added TP1: DONE, TestPoint:TestPoint_Pad_D1.0mm, symbol Connector:TestPoint
- added TP10: TMS, TestPoint:TestPoint_Pad_D1.0mm, symbol Connector:TestPoint
- added TP11: TDI, TestPoint:TestPoint_Pad_D1.0mm, symbol Connector:TestPoint
- added TP12: TDO, TestPoint:TestPoint_Pad_D1.0mm, symbol Connector:TestPoint
- added TP2: 5VSAT, TestPoint:TestPoint_Pad_D1.5mm, symbol Connector:TestPoint
- added TP3: 5VUSB, TestPoint:TestPoint_Pad_D1.5mm, symbol Connector:TestPoint
- added TP4: 5VSYS, TestPoint:TestPoint_Pad_D1.5mm, symbol Connector:TestPoint
- added TP5: 3.3V, TestPoint:TestPoint_Pad_D1.5mm, symbol Connector:TestPoint
- added TP6: TestPoint, TestPoint:TestPoint_Pad_D1.5mm, symbol Connector:TestPoint
- added TP7: 2.5V, TestPoint:TestPoint_Pad_D1.5mm, symbol Connector:TestPoint
- added TP8: TCK, TestPoint:TestPoint_Pad_D1.0mm, symbol Connector:TestPoint
- added TP9: 1.1V, TestPoint:TestPoint_Pad_D1.5mm, symbol Connector:TestPoint
- added U13, U18: W25Q16JVSS, Package_SO:SOIC-8_5.3x5.3mm_P1.27mm, symbol Memory_Flash:W25Q16JVSS
- added U15: XC6206PxxxMR, Package_TO_SOT_SMD:SOT-23-3, symbol Regulator_Linear:XC6206PxxxMR
- added U16: RP2040, Package_DFN_QFN:QFN-56-1EP_7x7mm_P0.4mm_EP3.2x3.2mm, symbol MCU_RaspberryPi:RP2040
- added U4: MT48LC16M16A2TG, Package_SO:TSOP-II-54_22.2x10.16mm_P0.8mm, symbol Memory_RAM:MT48LC16M16A2TG
- added Y1: Crystal_GND24, Crystal:Crystal_SMD_3225-4Pin_3.2x2.5mm, symbol Device:Crystal_GND24
- added Y2: SG-8002CE, Oscillator:Oscillator_SMD_SiT_PQFN-4Pin_2.5x2.0mm, symbol Oscillator:SG-8002CE
- C24: value 10uF -> 0.1uF; footprint Capacitor_SMD:C_1206_3216Metric_Pad1.33x1.80mm_HandSolder -> Capacitor_SMD:C_0603_1608Metric_Pad1.08x0.95mm_HandSolder
- renumbered U13 to CN4
Connections:
- net SDRAM_AUX_A0 is gone; now on net SDRAM2_A0: U3.23 (A0)
- net SDRAM_AUX_A1 is gone; now on net SDRAM2_A1: U3.24 (A1)
- net SDRAM_AUX_A10 is gone; now on net SDRAM2_A10: U3.22 (A10)
- net SDRAM_AUX_A11 is gone; now on net SDRAM2_A11: U3.35 (A11)
- net SDRAM_AUX_A12 is gone; now on net SDRAM2_A12: U3.36 (A12)
- net SDRAM_AUX_A2 is gone; now on net SDRAM2_A2: U3.25 (A2)
- net SDRAM_AUX_A3 is gone; now on net SDRAM2_A3: U3.26 (A3)
- net SDRAM_AUX_A4 is gone; now on net SDRAM2_A4: U3.29 (A4)
- net SDRAM_AUX_A5 is gone; now on net SDRAM2_A5: U3.30 (A5)
- net SDRAM_AUX_A6 is gone; now on net SDRAM2_A6: U3.31 (A6)
- net SDRAM_AUX_A7 is gone; now on net SDRAM2_A7: U3.32 (A7)
- net SDRAM_AUX_A8 is gone; now on net SDRAM2_A8: U3.33 (A8)
- net SDRAM_AUX_A9 is gone; now on net SDRAM2_A9: U3.34 (A9)
- net SDRAM_AUX_BA0 is gone; now on net SDRAM2_BA0: U3.20 (BA0)
- net SDRAM_AUX_BA1 is gone; now on net SDRAM2_BA1: U3.21 (BA1)
- net SDRAM_AUX_CAS is gone; now on net SDRAM2_CAS: U3.17 (~{CAS})
- net SDRAM_AUX_CKE is gone; now on net SDRAM2_CKE: U3.37 (CKE)
- net SDRAM_AUX_CLK is gone; now on net SDRAM2_CLK: U3.38 (CLK)
- net SDRAM_AUX_CS is gone; now on net SDRAM2_CS: U3.19 (~{CS})
- net SDRAM_AUX_DQ0 is gone; now on net SDRAM2_DQ0: U3.2 (DQ0)
- net SDRAM_AUX_DQ1 is gone; now on net SDRAM2_DQ1: U3.4 (DQ1)
- net SDRAM_AUX_DQ2 is gone; now on net SDRAM2_DQ2: U3.5 (DQ2)
- net SDRAM_AUX_DQ3 is gone; now on net SDRAM2_DQ3: U3.7 (DQ3)
- net SDRAM_AUX_DQ4 is gone; now on net SDRAM2_DQ4: U3.8 (DQ4)
- net SDRAM_AUX_DQ5 is gone; now on net SDRAM2_DQ5: U3.10 (DQ5)
- net SDRAM_AUX_DQ6 is gone; now on net SDRAM2_DQ6: U3.11 (DQ6)
- net SDRAM_AUX_DQ7 is gone; now on net SDRAM2_DQ7: U3.13 (DQ7)
- net SDRAM_AUX_DQM0 is gone; now on net SDRAM2_DQM0: U3.15 (DQML)
- net SDRAM_AUX_DQM1 is gone; now on net SDRAM2_DQM1: U3.39 (DQMH)
- net SDRAM_AUX_RAS is gone; now on net SDRAM2_RAS: U3.18 (~{RAS})
- net SDRAM_AUX_WE is gone; now on net SDRAM2_WE: U3.16 (~{WE})
- net +3_3V: now also C23.1, U6.F10 (VCCIO1), U6.F11 (VCCIO1), U6.F6 (VCCIO0), U6.F7 (VCCIO0), U6.H11 (VCCIO2), U6.H6 (VCCIO7), U6.H7 (VCCIO7), U6.J11 (VCCIO2), U6.J6 (VCCIO6), U6.J7 (VCCIO6), U6.K11 (VCCIO3), U6.L11 (VCCIO3), U6.L6 (VCCIO8), U6.P10 (CFG_1), C10.1, C11.1, C33.1, C34.1, C35.1, C36.1, C5.1, C56.1, C6.1, C60.1, C61.1, C62.1, C68.1, C7.1, C8.1, C9.1, R22.2, R23.1, R24.1, R25.1, R31.2, R32.2, R33.1, R34.1, R35.1, R36.1, R37.1, R38.1, U13.8 (VCC), U16.1 (IOVDD), U16.10 (IOVDD), U16.22 (IOVDD), U16.33 (IOVDD), U16.42 (IOVDD), U16.44 (VREG_VIN), U16.48 (USB_VDD), U16.49 (IOVDD), U18.8 (VCC), U4.1 (VDD), U4.14 (VDD), U4.27 (VDD), U4.3 (VDDQ), U4.43 (VDDQ), U4.49 (VDDQ), U4.9 (VDDQ), Y2.4 (Vcc)
- net +5V_SATURN: now also TP2.1
- net +5V_SYS: now also U14.1 (EN), U14.4 (IN), U7.1 (EN), U7.4 (IN), C27.1, C66.1, C67.1, TP4.1, U15.3 (VI); no longer C23.1
- net 5V_SATURN_DETECT: now also U6.J13 (PR17C)
- net ABUS_3V_A1: now also U6.J14 (PR20C)
- net ABUS_3V_A10: now also U6.K14 (PR20D)
- net ABUS_3V_A11: now also U6.L14 (PR32C)
- net ABUS_3V_A12: now also U6.P11 (PR47C)
- net ABUS_3V_A13: now also U6.N12 (PR44D)
- net ABUS_3V_A14: now also U6.R3 (PL41B)
- net ABUS_3V_A15: now also U6.N6 (PL47B)
- net ABUS_3V_A16: now also U6.T2 (PL38D)
- net ABUS_3V_A17: now also U6.N5 (PL44D)
- net ABUS_3V_A18: now also U6.P3 (PL38B)
- net ABUS_3V_A19: now also U6.P4 (PL41A)
- net ABUS_3V_A2: now also U6.T6 (PB4A)
- net ABUS_3V_A20: now also U6.R2 (PL38C)
- net ABUS_3V_A21: now also U6.N4 (PL38A)
- net ABUS_3V_A22: now also U6.R1 (PL35B)
- net ABUS_3V_A23: now also U6.M4 (PL35C)
- net ABUS_3V_A24: now also U6.P2 (PL32B)
- net ABUS_3V_A3: now also U6.P5 (PL47D)
- net ABUS_3V_A4: now also U6.R5 (PL44A)
- net ABUS_3V_A5: now also U6.T4 (PL44B)
- net ABUS_3V_A6: now also U6.R4 (PL41C)
- net ABUS_3V_A7: now also U6.T3 (PL41D)
- net ABUS_3V_A8: now also U6.N13 (PR38A)
- net ABUS_3V_A9: now also U6.L13 (PR29C)
- net ABUS_3V_CS0: now also U6.H14 (PR14D)
- net ABUS_3V_CS1: now also U6.R7 (PB6A)
- net ABUS_3V_CS2: now also U6.G14 (PR14C)
- net ABUS_3V_D0: now also U6.E13 (PT62B)
- net ABUS_3V_D1: now also U6.D14 (PR2D)
- net ABUS_3V_D10: now also U6.T13 (PR44B)
- net ABUS_3V_D11: now also U6.P13 (PR41A)
- net ABUS_3V_D12: now also U6.P16 (PR35A)
- net ABUS_3V_D13: now also U6.P15 (PR32B)
- net ABUS_3V_D14: now also U6.R16 (PR35B)
- net ABUS_3V_D15: now also U6.P14 (PR38B)
- net ABUS_3V_D2: now also U6.C13 (PT60B)
- net ABUS_3V_D3: now also U6.R12 (PR44A)
- net ABUS_3V_D4: now also U6.R15 (PR38C)
- net ABUS_3V_D5: now also U6.T15 (PR38D)
- net ABUS_3V_D6: now also U6.R14 (PR41B)
- net ABUS_3V_D7: now also U6.T14 (PR41D)
- net ABUS_3V_D8: now also U6.P12 (PR47D)
- net ABUS_3V_D9: now also U6.R13 (PR41C)
- net ABUS_3V_IRQ: now also U6.J3 (PL20C)
- net ABUS_3V_MUX_DATA_DIR: now also U6.H4 (PL17B)
- net ABUS_3V_RD: now also U6.R6 (PB4B)
- net ABUS_3V_WR0: now also U6.F14 (PR5D)
- net ABUS_3V_WR1: now also U6.R8 (PB13A)
- net BUFFERS_OE: now also U6.L3 (PL32C)
- net ESP32_CS: now also U6.C6 (PT22A)
- net ESP32_MISO: now also U6.E7 (PT24A)
- net ESP32_MOSI: now also U6.D6 (PT20B)
- net ESP32_SCK: now also U6.C7 (PT27A)
- net GND: now also U14.2 (GND), U6.N10 (CFG_0), U6.R10 (CFG_2), U7.2 (GND), C10.2, C11.2, C12.2, C13.2, C14.2, C15.2, C16.2, C18.2, C19.2, C20.1, C27.2, C28.2, C30.2, C32.2, C33.2, C34.2, C35.2, C36.2, C5.2, C56.2, C57.2, C58.2, C59.2, C6.2, C60.2, C61.2, C62.2, C66.2, C67.2, C68.2, C7.2, C8.2, C9.2, CN3.A1 (GND), CN3.A12 (GND), CN3.B1 (GND), CN3.B12 (GND), CN3.SH (SHIELD), D3.1 (K), R12.2, R13.2, R27.1, R29.1, R6.1, SW1.1, SW2.1, U13.4 (GND), U15.1 (GND), U16.19 (TESTEN), U16.57 (GND), U18.4 (GND), U4.12 (VSSQ), U4.28 (VSS), U4.41 (VSS), U4.46 (VSSQ), U4.52 (VSSQ), U4.54 (VSS), U4.6 (VSSQ), Y1.2 (G), Y1.4 (G), Y2.2 (GND); no longer U2.2 (1B0)
- net IBCK_3V: now also U6.F4 (PL8C)
- net ILRCK_3V: now also U6.P8 (PB13B)
- net IRQ_OUT_ENABLE: now also U6.F3 (PL5D)
- net ISD_3V: now also U6.E3 (PL5C)
- net LEDB: now also U6.D7 (PT24B)
- net LEDG: now also U6.E8 (PT33A)
- net LEDR: now also U6.E9 (PT40B)
- net RESET_3V: now also U6.K4 (PL29A)
- net SCSPCLK: now also U2.2 (1B0)
- net SD_CLK: now also U6.E11 (PT51B)
- net SD_CMD: now also U6.C9 (PT38B)
- net SD_DAT0: now also U6.C11 (PT49B)
- net SD_DAT1: now also U6.D12 (PT58A)
- net SD_DAT2: now also U6.D8 (PT33B)
- net SD_DAT3: now also U6.D10 (PT47A)
- net SD_DET_A: now also U6.C12 (PT56B)
- net SD_DET_B: now also U6.E10 (PT47B)
- net SSEL_3V: now also U6.D4 (PT9B)
- net SCSPCLK_3V: now reaches U2.47 (1A0)
- net SCSPCLK_3V: now also U6.G3 (PL14C)
- net +5V_USB: now reaches D4.2
- net +5V_USB: now also C18.1, CN3.A4 (VBUS), CN3.A9 (VBUS), CN3.B4 (VBUS), CN3.B9 (VBUS), TP3.1
- net at U14.3 (LX): now also L2.1
- net at U14.5 (FB): now also C31.2, R28.2, R29.2
- net SDRAM1_A3: now reaches U6.A10 (PT42B)
- net SDRAM1_A3: now also U4.26 (A3)
- net SDRAM1_BA1: now reaches U6.A11 (PT53A)
- net SDRAM1_BA1: now also U4.21 (BA1)
- net SDRAM1_CS: now reaches U6.A12 (PT53B)
- net SDRAM1_CS: now also U4.19 (~{CS})
- net SDRAM1_CAS: now reaches U6.A13 (PT65A)
- net SDRAM1_CAS: now also U4.17 (~{CAS})
- net SDRAM1_DQM0: now reaches U6.A14 (PT65B)
- net SDRAM1_DQM0: now also U4.15 (DQML)
- net SDRAM1_DQ6: now reaches U6.A15 (PT67B)
- net SDRAM1_DQ6: now also U4.11 (DQ6)
- net SDRAM2_A11: now reaches U6.A5 (PT18A)
- net SDRAM2_A8: now reaches U6.A6 (PT18B)
- net SDRAM2_A5: now reaches U6.A7 (PT29A)
- net SDRAM2_A7: now reaches U6.A8 (PT29B)
- net SDRAM1_A1: now reaches U6.A9 (PT42A)
- net SDRAM1_A1: now also U4.24 (A1)
- net SDRAM1_A10: now reaches U6.B10 (PT44A)
- net SDRAM1_A10: now also U4.22 (A10)
- net SDRAM1_BA0: now reaches U6.B11 (PT49A)
- net SDRAM1_BA0: now also U4.20 (BA0)
- net SDRAM1_RAS: now reaches U6.B12 (PT56A)
- net SDRAM1_RAS: now also U4.18 (~{RAS})
- net SDRAM1_WE: now reaches U6.B13 (PT60A)
- net SDRAM1_WE: now also U4.16 (~{WE})
- net SDRAM1_DQ7: now reaches U6.B14 (PT67A)
- net SDRAM1_DQ7: now also U4.13 (DQ7)
- net SDRAM2_A4: now reaches U6.B6 (PT22B)
- net SDRAM2_A6: now reaches U6.B7 (PT27B)
- net SDRAM1_A0: now reaches U6.B8 (PT35B)
- net SDRAM1_A0: now also U4.23 (A0)
- net SDRAM1_A2: now reaches U6.B9 (PT38A)
- net SDRAM1_A2: now also U4.25 (A2)
- net SDRAM2_DQ9: now reaches U6.A2 (PT4A)
- net SDRAM2_DQ9: now also U3.44 (DQ9)
- net SDRAM2_DQM1: now reaches U6.A3 (PT6A)
- net SDRAM2_CKE: now reaches U6.A4 (PT6B)
- net SDRAM1_DQ4: now reaches U6.B15 (PR2B)
- net SDRAM1_DQ4: now also U4.8 (DQ4)
- net SDRAM1_DQ3: now reaches U6.B16 (PR2A)
- net SDRAM1_DQ3: now also U4.7 (DQ3)
- net SDRAM2_DQ10: now reaches U6.B3 (PT4B)
- net SDRAM2_DQ10: now also U3.45 (DQ10)
- net SDRAM2_CLK: now reaches U6.B4 (PT11B)
- net SDRAM2_A9: now reaches U6.B5 (PT15B)
- net SDRAM1_DQ5: now reaches U6.C14 (PR2C)
- net SDRAM1_DQ5: now also U4.10 (DQ5)
- net SDRAM1_DQ2: now reaches U6.C15 (PR5B)
- net SDRAM1_DQ2: now also U4.5 (DQ2)
- net SDRAM1_DQ1: now reaches U6.C16 (PR5A)
- net SDRAM1_DQ1: now also U4.4 (DQ1)
- net SDRAM2_DQ8: now reaches U6.C4 (PT11A)
- net SDRAM2_DQ8: now also U3.42 (DQ8)
- net SDRAM2_A12: now reaches U6.C5 (PT15A)
- net SDRAM1_DQ15: now reaches U6.D16 (PR8A)
- net SDRAM1_DQ15: now also U4.53 (DQ15)
- net SDRAM1_DQ0: now reaches U6.E14 (PR5C)
- net SDRAM1_DQ0: now also U4.2 (DQ0)
- net SDRAM1_DQ14: now reaches U6.E15 (PR8B)
- net SDRAM1_DQ14: now also U4.51 (DQ14)
- net SDRAM1_DQ13: now reaches U6.E16 (PR11D)
- net SDRAM1_DQ13: now also U4.50 (DQ13)
- net SDRAM1_DQ12: now reaches U6.F15 (PR11C)
- net SDRAM1_DQ12: now also U4.48 (DQ12)
- net SDRAM1_DQ11: now reaches U6.F16 (PR14A)
- net SDRAM1_DQ11: now also U4.47 (DQ11)
- net SDRAM1_DQ10: now reaches U6.G15 (PR14B)
- net SDRAM1_DQ10: now also U4.45 (DQ10)
- net SDRAM1_DQ9: now reaches U6.G16 (PR20A)
- net SDRAM1_DQ9: now also U4.44 (DQ9)
- net SDRAM1_DQ8: now reaches U6.H15 (PR20B)
- net SDRAM1_DQ8: now also U4.42 (DQ8)
- net SDRAM1_DQM1: now reaches U6.J15 (PR23B)
- net SDRAM1_DQM1: now also U4.39 (DQMH)
- net SDRAM1_A4: now reaches U6.J16 (PR23A)
- net SDRAM1_A4: now also U4.29 (A4)
- net SDRAM1_A5: now reaches U6.K15 (PR23D)
- net SDRAM1_A5: now also U4.30 (A5)
- net SDRAM1_A6: now reaches U6.K16 (PR23C)
- net SDRAM1_A6: now also U4.31 (A6)
- net SDRAM1_A7: now reaches U6.L15 (PR26B)
- net SDRAM1_A7: now also U4.32 (A7)
- net SDRAM1_A8: now reaches U6.L16 (PR26A)
- net SDRAM1_A8: now also U4.33 (A8)
- net SDRAM1_A9: now reaches U6.M14 (PR32D)
- net SDRAM1_A9: now also U4.34 (A9)
- net SDRAM1_A12: now reaches U6.M15 (PR26D)
- net SDRAM1_A12: now also U4.36 (A12)
- net SDRAM1_A11: now reaches U6.M16 (PR26C)
- net SDRAM1_A11: now also U4.35 (A11)
- net SDRAM1_CLK: now reaches U6.N14 (PR35D)
- net SDRAM1_CLK: now also U4.38 (CLK)
- net SDRAM1_CKE: now reaches U6.N16 (PR32A)
- net SDRAM1_CKE: now also U4.37 (CKE)
- net CLK_25M: now reaches U6.P6 (PL47C)
- net CLK_25M: now also Y2.3 (OUT)
- net SDRAM2_DQ11: now reaches U3.47 (DQ11)
- net SDRAM2_DQ11: now also U6.B2 (PL2B)
- net SDRAM2_DQ12: now reaches U3.48 (DQ12)
- net SDRAM2_DQ12: now also U6.B1 (PL2A)
- net SDRAM2_DQ13: now reaches U3.50 (DQ13)
- net SDRAM2_DQ13: now also U6.C3 (PL2C)
- net SDRAM2_DQ14: now reaches U3.51 (DQ14)
- net SDRAM2_DQ14: now also U6.C1 (PL5A)
- net SDRAM2_DQ15: now reaches U3.53 (DQ15)
- net SDRAM2_DQ15: now also U6.C2 (PL5B)
- net at U7.3 (LX): now also L1.1
- net at U7.5 (FB): now also C29.2, R26.2, R27.2
- net SDRAM2_DQ0: now reaches U6.D1 (PL8A)
- net SDRAM2_DQ1: now reaches U6.D3 (PL2D)
- net SDRAM2_DQ2: now reaches U6.E1 (PL11D)
- net SDRAM2_DQ3: now reaches U6.E2 (PL8B)
- net SDRAM2_DQ4: now reaches U6.F1 (PL14A)
- net SDRAM2_DQ5: now reaches U6.F2 (PL11C)
- net SDRAM2_DQ6: now reaches U6.G1 (PL20A)
- net SDRAM2_DQ7: now reaches U6.G2 (PL14B)
- net SDRAM2_A3: now reaches U6.H2 (PL20B)
- net SDRAM2_A2: now reaches U6.J1 (PL23A)
- net SDRAM2_A1: now reaches U6.J2 (PL23B)
- net SDRAM2_A0: now reaches U6.K1 (PL23C)
- net SDRAM2_A10: now reaches U6.K2 (PL23D)
- net SDRAM2_BA1: now reaches U6.L1 (PL26A)
- net SDRAM2_BA0: now reaches U6.L2 (PL26B)
- net SDRAM2_CS: now reaches U6.M1 (PL26C)
- net JTAG_TDO: now reaches U6.M10 (TDO)
- net JTAG_TDO: now also TP12.1
- net SDRAM2_RAS: now reaches U6.M2 (PL26D)
- net FPGA_QSPI_D2: now reaches U6.M7 (PB9B)
- net FPGA_QSPI_D2: now also R37.2, U16.3 (GPIO1), U18.3 (~{WP}/IO_{2})
- net SDRAM2_CAS: now reaches U6.N1 (PL32A)
- net SDRAM2_WE: now reaches U6.N3 (PL35D)
- net FPGA_QSPI_D3: now reaches U6.N7 (PB9A)
- net FPGA_QSPI_D3: now also R38.2, U16.12 (GPIO9), U18.7 (~{HOLD}/~{RESET}/IO_{3})
- net FPGA_QSPI_CS: now reaches U6.N8 (PB15A)
- net FPGA_QSPI_CS: now also R33.2, U16.5 (GPIO3), U18.1 (~{CS})
- net FPGA_QSPI_CLK: now reaches U6.N9 (CCLK)
- net FPGA_QSPI_CLK: now also R34.2, U16.9 (GPIO7), U18.6 (CLK)
- net SDRAM2_DQM0: now reaches U6.P1 (PL35A)
- net at U6.P9 (DONE): now also R30.2, R31.1, TP1.1
- net JTAG_TDI: now reaches U6.R11 (TDI)
- net JTAG_TDI: now also TP11.1
- net PROGRAMN: now reaches U6.R9 (PROGRAMN)
- net PROGRAMN: now also R24.2, SW2.2, U16.29 (GPIO18)
- net JTAG_TCK: now reaches U6.T10 (TCK)
- net JTAG_TCK: now also R6.2, TP8.1
- net JTAG_TMS: now reaches U6.T11 (TMS)
- net JTAG_TMS: now also TP10.1
- net FPGA_QSPI_D1: now reaches U6.T7 (PB11A)
- net FPGA_QSPI_D1: now also R36.2, U16.14 (GPIO11), U18.2 (DO/IO_{1})
- net FPGA_QSPI_D0: now reaches U6.T8 (PB11B)
- net FPGA_QSPI_D0: now also R35.2, U16.7 (GPIO5), U18.5 (DI/IO_{0})
- net at U6.T9 (INITN): now also R23.2
- net +2_5V: now reaches U6.G11 (VCCAUX)
- net +2_5V: now also U6.L7 (VCCAUX), C15.1, C16.1, R40.2
- net +1_1V: now reaches U6.G6 (VCC)
- net +1_1V: now also U6.G7 (VCC), U6.G9 (VCC), U6.L10 (VCC), U6.L8 (VCC), U6.L9 (VCC), C12.1, C13.1, C14.1, R39.2
- new net: R22.1, U16.43 (ADC_AVDD)
- new net: C28.1, R40.1, TP7.1, U15.2 (VO)
- new net: CN3.B5 (CC2), R13.1
- new net: C31.1, C32.1, L2.2, R28.1, R39.1, TP9.1
- new net: C29.1, C30.1, L1.2, R26.1, R32.1, TP5.1
- new net: C20.2, U16.21 (XOUT), Y1.1
- new net: R25.2, Y2.1 (OE)
- new net: D3.2 (A), R30.1
- new net: C19.1, U16.20 (XIN), Y1.3
- new net: CN3.A5 (CC1), R12.1
- new net: R20.1, SW1.2
- new net: R18.2, U16.47 (USB_DP)
- new net: R14.2, U16.46 (USB_DM)
- new net +1_1V_RPI: C57.1, C58.1, C59.1, TP6.1, U16.23 (DVDD), U16.45 (VREG_VOUT), U16.50 (DVDD)
- new net RP_QSPI_CLK: U13.6 (CLK), U16.52 (QSPI_SCLK)
- new net RP_QSPI_CS: R20.2, U13.1 (~{CS}), U16.56 (~{QSPI_SS})
- new net RP_QSPI_D0: U13.5 (DI/IO_{0}), U16.53 (QSPI_SD0)
- new net RP_QSPI_D1: U13.2 (DO/IO_{1}), U16.55 (QSPI_SD1)
- new net RP_QSPI_D2: U13.3 (~{WP}/IO_{2}), U16.54 (QSPI_SD2)
- new net RP_QSPI_D3: U13.7 (~{HOLD}/~{RESET}/IO_{3}), U16.51 (QSPI_SD3)
- new net USB_DM: CN3.A7 (D-), CN3.B7 (D-), R14.1
- new net USB_DP: CN3.A6 (D+), CN3.B6 (D+), R18.1
Other:
- note added: "Compatible connectors: JAE DX07S016JA1R1500 JAE DX07S016JA3R1500 HROPARTS TYPE-C-31-M-12 HROPARTS TYPE-C-31-M-14 XKB U262-161N-4BVC11 Jing Ext. C167321"
- note added: "PROGRAM PICO"
- note removed: "External 5V power supply + 3V3 power output/check"
- note removed: "MFG P/N : 1473005-4 1565917-4"
- note removed: "SDRAM : shares 3V3 with MAX10 DDR : requires 2V5 power supply"
- moved on the sheet: C39, C4, C54, C55, CN2, CN4, CN5, D4, R15, R16, R17, R8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

Commit message: Board rerouting
Parts:
- C1: renamed from C43; LCSC (none) -> C1590
- C10: renamed from C47; LCSC (none) -> C1590
- C11: renamed from C51; LCSC (none) -> C1590
- C12: renamed from C19; LCSC (none) -> C1644
- C13: renamed from C20; LCSC (none) -> C1644
- C14: renamed from C22; LCSC (none) -> C1590
- C15: renamed from C26; LCSC (none) -> C1590
- C16: renamed from C2; LCSC (none) -> C1590
- C17: renamed from C44; LCSC (none) -> C1590
- C18: renamed from C46; LCSC (none) -> C1590
- C19: renamed from C50; LCSC (none) -> C1590
- C2: renamed from C49; LCSC (none) -> C1590
- C20: renamed from C60; LCSC (none) -> C1590
- C21: renamed from C61; LCSC (none) -> C1590
- C22: renamed from C57; LCSC (none) -> C1590
- C23: renamed from C62; LCSC (none) -> C1590
- C24: renamed from C58; LCSC (none) -> C1590
- C25: renamed from C21; LCSC (none) -> C1590
- C26: renamed from C59; LCSC (none) -> C1590
- C27: renamed from C1; LCSC (none) -> C1590
- C28: renamed from C25; LCSC (none) -> C1590
- C29: renamed from C54; LCSC (none) -> C1705
- C3: LCSC (none) -> C1705
- C30: renamed from C66; LCSC (none) -> C59461
- C31: renamed from C67; LCSC (none) -> C59461
- C32: renamed from C27; LCSC (none) -> C1592
- C33: renamed from C5; LCSC (none) -> C1590
- C34: renamed from C4; LCSC (none) -> C1590
- C35: renamed from C23; LCSC (none) -> C1590
- C36: renamed from C33; LCSC (none) -> C1590
- C37: renamed from C24; LCSC (none) -> C1590
- C38: renamed from C34; LCSC (none) -> C1590
- C39: renamed from C35; LCSC (none) -> C1590
- C4: renamed from C42; LCSC (none) -> C1590
- C40: renamed from C36; LCSC (none) -> C1590
- C41: renamed from C28; LCSC (none) -> C1592
- C42: renamed from C29; LCSC (none) -> C1647
- C43: renamed from C31; LCSC (none) -> C1647
- C44: renamed from C30; LCSC (none) -> C1691
- C45: renamed from C32; LCSC (none) -> C1691
- C46: renamed from C39; LCSC (none) -> C1590
- C47: renamed from C55; LCSC (none) -> C1590
- C48: renamed from C68; LCSC (none) -> C1590
- C49: renamed from C15; LCSC (none) -> C1525
- C5: renamed from C48; LCSC (none) -> C1590
- C50: renamed from C16; LCSC (none) -> C1525
- C51: renamed from C11; LCSC (none) -> C1525
- C52: renamed from C10; LCSC (none) -> C1525
- C53: renamed from C9; LCSC (none) -> C1525
- C54: renamed from C12; LCSC (none) -> C1525
- C55: renamed from C8; LCSC (none) -> C1525
- C56: renamed from C13; LCSC (none) -> C1525
- C57: renamed from C7; LCSC (none) -> C1525
- C58: renamed from C14; LCSC (none) -> C1525
- C59: renamed from C6; LCSC (none) -> C1525
- C6: renamed from C18; LCSC (none) -> C1705
- C7: renamed from C56; LCSC (none) -> C1590
- C8: renamed from C17; LCSC (none) -> C1705
- C9: renamed from C45; LCSC (none) -> C1590
- CN1: renamed from CN3; LCSC (none) -> C3197885
- CN2: renamed from CN1; now left out of the parts list
- CN3: renamed from CN2; now not fitted; now left out of the parts list
- CN4: renamed from CN5; LCSC (none) -> C266602
- CN5: renamed from CN4; LCSC (none) -> C27438
- D1: renamed from D4; LCSC (none) -> C2135
- D2: now not fitted; now left out of the parts list
- D3: renamed from D1; LCSC (none) -> C7371892
- D4: renamed from D3; LCSC (none) -> C965863
- KICAD1, SEGATA1, SHIRO!1, SW1, TP12, TP2, VACHE1: now left out of the parts list
- L1, L2: LCSC (none) -> C86092
- R1: renamed from R12; LCSC (none) -> C23186
- R10: renamed from R28; LCSC (none) -> C25811
- R11: renamed from R10; LCSC (none) -> C23179
- R12: renamed from R27; LCSC (none) -> C22807
- R13: renamed from R29; LCSC (none) -> C4197
- R14: renamed from R11; LCSC (none) -> C23179
- R15: renamed from R19; LCSC (none) -> C23179
- R16: renamed from R32; LCSC (none) -> C21189
- R17: renamed from R39; LCSC (none) -> C21189
- R18: renamed from R6; LCSC (none) -> C23162
- R19: renamed from R31; LCSC (none) -> C21190
- R2: renamed from R20; LCSC (none) -> C21190
- R20: renamed from R30; LCSC (none) -> C21190
- R21: renamed from R24; LCSC (none) -> C25804
- R22: renamed from R23; LCSC (none) -> C25804
- R23: renamed from R8; LCSC (none) -> C4216
- R24: renamed from R9; LCSC (none) -> C4216
- R25: renamed from R15; LCSC (none) -> C4216
- R26: renamed from R16; LCSC (none) -> C4216
- R27: renamed from R17; LCSC (none) -> C4216
- R28: renamed from R25; LCSC (none) -> C21189
- R29: renamed from R33; LCSC (none) -> C25804
- R3: renamed from R21; LCSC (none) -> C21189
- R30: renamed from R34; LCSC (none) -> C25804
- R31: renamed from R35; LCSC (none) -> C25804
- R32: renamed from R36; LCSC (none) -> C25804
- R33: renamed from R37; LCSC (none) -> C25804
- R34: renamed from R38; LCSC (none) -> C25804
- R35: renamed from R4; LCSC (none) -> C23162
- R36: renamed from R5; LCSC (none) -> C25804
- R4: renamed from R13; LCSC (none) -> C23186
- R5: renamed from R14; LCSC (none) -> C25190
- R6: renamed from R18; LCSC (none) -> C25190
- R7: renamed from R22; LCSC (none) -> C21189
- R8: renamed from R40; LCSC (none) -> C21189
- R9: renamed from R26; LCSC (none) -> C2907061
- SW2: footprint (none) -> Button_Switch_SMD:SW_SPST_EVQP2_ShortPushTravel_H2.5mm; now left out of the parts list
- TP1: renamed from TP6; now left out of the parts list
- TP10: renamed from TP11; now left out of the parts list
- TP11: renamed from TP10; now left out of the parts list
- TP3: renamed from TP4; now left out of the parts list
- TP4: renamed from TP3; now left out of the parts list
- TP5: renamed from TP7; now left out of the parts list
- TP6: renamed from TP5; now left out of the parts list
- TP7: renamed from TP9; now left out of the parts list
- TP8: renamed from TP1; now left out of the parts list
- TP9: renamed from TP8; now left out of the parts list
- U1: renamed from U8; LCSC (none) -> C7843
- U10: renamed from U1; LCSC (none) -> C53436298
- U11: renamed from U4; LCSC (none) -> C62246
- U12: renamed from U3; LCSC (none) -> C62246
- U13: renamed from U7; LCSC (none) -> C81889
- U14: LCSC (none) -> C81889
- U15: LCSC (none) -> C15906
- U16: renamed from U6; LCSC (none) -> C1521614
- U17: renamed from U18; LCSC (none) -> C82317
- U2: renamed from U11; LCSC (none) -> C7843
- U3: renamed from U13; LCSC (none) -> C82317
- U4: renamed from U9; LCSC (none) -> C7843
- U5: renamed from U10; LCSC (none) -> C7843
- U6: renamed from U12; LCSC (none) -> C7843
- U7: renamed from U2; LCSC (none) -> C53436298
- U8: renamed from U5; LCSC (none) -> C53436298
- U9: renamed from U16; LCSC (none) -> C2040
- Y1: LCSC (none) -> C9002
- Y2: LCSC (none) -> C49207939

Commit message: Board rerouting
Parts:
- CN2, KICAD1, SEGATA1, SHIRO!1, TP1, TP10, TP11, TP12, TP2, TP3, TP4, TP5, TP6, TP7, TP8, TP9, VACHE1: now not fitted
- SW1, SW2: now in the parts list
Changed lines of the file:
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@@
 		(on_board yes)
 		(in_pos_files yes)
-		(dnp no)
+		(dnp yes)
 		(property "Reference" "SEGATA1"
 			(at 387.35 114.2238 0)
@@
 		(on_board yes)
 		(in_pos_files yes)
-		(dnp no)
+		(dnp yes)
 		(property "Reference" "KICAD1"
 			(at 431.2412 181.7116 0)
@@
 		(on_board yes)
 		(in_pos_files yes)
-		(dnp no)
+		(dnp yes)
 		(property "Reference" "VACHE1"
 			(at 461.01 97.4344 0)
@@
 		(on_board yes)
 		(in_pos_files yes)
-		(dnp no)
+		(dnp yes)
 		(fields_autoplaced yes)
 		(property "Reference" "TP8"
@@
 		(on_board yes)
 		(in_pos_files yes)
-		(dnp no)
+		(dnp yes)
 		(fields_autoplaced yes)
 		(property "Reference" "CN2"
@@
 		(on_board yes)
 		(in_pos_files yes)
-		(dnp no)
+		(dnp yes)
 		(property "Reference" "TP4"
 			(at 457.2 519.43 90)
@@
 		(on_board yes)
 		(in_pos_files yes)
-		(dnp no)
+		(dnp yes)
 		(property "Reference" "SHIRO!1"
 			(at 426.72 151.13 0)
@@
 		(on_board yes)
 		(in_pos_files yes)
-		(dnp no)
+		(dnp yes)
 		(property "Reference" "TP7"
 			(at 547.37 591.058 90)
@@
 		(on_board yes)
 		(in_pos_files yes)
-		(dnp no)
+		(dnp yes)
 		(property "Reference" "TP10"
 			(at 656.59 75.184 90)
@@
 		(on_board yes)
 		(in_pos_files yes)
-		(dnp no)
+		(dnp yes)
 		(property "Reference" "TP11"
 			(at 656.59 77.724 90)
@@
 		(body_style 1)
 		(exclude_from_sim no)
-		(in_bom no)
+		(in_bom yes)
 		(on_board yes)
 		(in_pos_files yes)
@@
 		(on_board yes)
 		(in_pos_files yes)
-		(dnp no)
+		(dnp yes)
 		(property "Reference" "TP9"
 			(at 657.86 72.39 90)
@@
 		(on_board yes)
 		(in_pos_files yes)
-		(dnp no)
+		(dnp yes)
 		(fields_autoplaced yes)
 		(property "Reference" "TP1"
@@
 		(on_board yes)
 		(in_pos_files yes)
-		(dnp no)
+		(dnp yes)
 		(property "Reference" "TP3"
 			(at 398.78 528.066 90)
@@
 		(on_board yes)
 		(in_pos_files yes)
-		(dnp no)
+		(dnp yes)
 		(property "Reference" "TP5"
 			(at 495.3 555.498 90)
@@
 		(body_style 1)
 		(exclude_from_sim no)
-		(in_bom no)
+		(in_bom yes)
 		(on_board yes)
 		(in_pos_files yes)
@@
 		(on_board yes)
 		(in_pos_files yes)
-		(dnp no)
+		(dnp yes)
 		(property "Reference" "TP12"
 			(at 760.73 54.356 90)
@@
 		(on_board yes)
 		(in_pos_files yes)
-		(dnp no)
+		(dnp yes)
 		(property "Reference" "TP6"
 			(at 547.37 522.478 90)
@@
 		(on_board yes)
 		(in_pos_files yes)
-		(dnp no)
+		(dnp yes)
 		(property "Reference" "TP2"
 			(at 395.986 519.684 90)

Commit message: Cleanup gerber products
Parts:
- CN1: value USB_C_Receptacle_USB2.0_16P -> UC09-0B16F00P11; LCSC C3197885 -> C36936538
- CN4: value 693063020911 -> SD-CARD 11P; LCSC C266602 -> C7529393
- CN5: value ESP32_CAM_HALF -> 2.54-1*8P母环保
- R21, R22, R29, R30, R31, R32, R33, R34, R36: LCSC C25804 -> C15401
- SW1, SW2: value SW_Push -> TS-1101-C-W; footprint Button_Switch_SMD:SW_SPST_EVQP2_ShortPushTravel_H2.5mm -> Button_Switch_SMD:SW_Tactile_SPST_NO_Straight_CK_PTS636Sx25SMTRLFS; LCSC (none) -> C318938
- U1, U2, U4, U5, U6: value SN74LVC1T45DBV -> SN74LVC1T45DBVR
- U10, U7, U8: value 74ALVC164245 -> 74ALVC164245DGG:11-JSM
- U11, U12: value MT48LC16M16A2TG -> W9825G6KH-6
- U15: value XC6206PxxxMR -> XC6206P252MR
- U17, U3: value W25Q16JVSS -> P25Q16SH-SSH-IR; LCSC C82317 -> C7466814
- Y1: value Crystal_GND24 -> X322512MSB4SI
- Y2: value SG-8002CE -> SX2M25.000M20F30TNN; LCSC C49207939 -> C2901601
Changed lines of the file:
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@@
 			)
 		)
-		(property "Value" "74ALVC164245"
+		(property "Value" "74ALVC164245DGG:11-JSM"
 			(at 223.52 260.35 0)
 			(show_name no)
@@
 			)
 		)
-		(property "Value" "74ALVC164245"
+		(property "Value" "74ALVC164245DGG:11-JSM"
 			(at 223.52 134.62 0)
 			(show_name no)
@@
 			)
 		)
-		(property "Value" "74ALVC164245"
+		(property "Value" "74ALVC164245DGG:11-JSM"
 			(at 247.65 34.29 0)
 			(show_name no)
@@
 			)
 		)
-		(property "Value" "ESP32_CAM_HALF"
+		(property "Value" "2.54-1*8P母环保"
 			(at 985.012 540.258 0)
 			(show_name no)
@@
 			)
 		)
-		(property "Value" "SN74LVC1T45DBV"
+		(property "Value" "SN74LVC1T45DBVR"
 			(at 81.28 396.24 0)
 			(show_name no)
@@
 			)
 		)
-		(property "Value" "SN74LVC1T45DBV"
+		(property "Value" "SN74LVC1T45DBVR"
 			(at 68.58 438.15 0)
 			(show_name no)
@@
 			)
 		)
-		(property "Value" "SN74LVC1T45DBV"
+		(property "Value" "SN74LVC1T45DBVR"
 			(at 177.8 393.7 0)
 			(show_name no)
@@
 			)
 		)
-		(property "Value" "SN74LVC1T45DBV"
+		(property "Value" "SN74LVC1T45DBVR"
 			(at 177.8 430.53 0)
 			(show_name no)
@@
 			)
 		)
-		(property "Value" "SN74LVC1T45DBV"
+		(property "Value" "SN74LVC1T45DBVR"
 			(at 177.8 466.09 0)
 			(show_name no)
@@
 			)
 		)
-		(property "LCSC" "C25804"
+		(property "LCSC" " C15401"
 			(at 668.02 67.31 90)
 			(hide yes)
@@
 			)
 		)
-		(property "Value" "XC6206PxxxMR"
+		(property "Value" "XC6206P252MR"
 			(at 471.17 557.53 0)
 			(show_name no)
@@
 			)
 		)
-		(property "LCSC" "C25804"
+		(property "LCSC" " C15401"
 			(at 934.72 295.91 90)
 			(hide yes)
@@
 			)
 		)
-		(property "Value" "W25Q16JVSS"
+		(property "Value" "P25Q16SH-SSH-IR"
 			(at 981.71 292.0999 0)
 			(show_name no)
@@
 			)
 		)
-		(property "LCSC" "C82317"
+		(property "LCSC" "C7466814"
 			(at 970.28 290.83 0)
 			(hide yes)
@@
 			)
 		)
-		(property "Value" "MT48LC16M16A2TG"
+		(property "Value" "W9825G6KH-6"
 			(at 430.1333 275.59 0)
 			(show_name no)
@@
 			)
 		)
-		(property "LCSC" "C25804"
+		(property "LCSC" " C15401"
 			(at 1115.06 102.87 90)
 			(hide yes)
@@
 			)
 		)
-		(property "LCSC" "C25804"
+		(property "LCSC" " C15401"
 			(at 934.72 293.37 90)
 			(hide yes)
@@
 			)
 		)
-		(property "Value" "MT48LC16M16A2TG"
+		(property "Value" "W9825G6KH-6"
 			(at 430.0094 372.11 0)
 			(show_name no)
@@
 			)
 		)
-		(property "Value" "Crystal_GND24"
+		(property "Value" "X322512MSB4SI"
 			(at 181.61 612.1399 90)
 			(show_name no)
@@
 			)
 		)
-		(property "Value" "SG-8002CE"
+		(property "Value" "SX2M25.000M20F30TNN"
 			(at 802.64 257.7398 0)
 			(show_name no)
@@
 			)
 		)
-		(property "LCSC" "C49207939"
+		(property "LCSC" "C2901601"
 			(at 789.94 261.62 0)
 			(hide yes)
@@
 			)
 		)
-		(property "LCSC" "C25804"
+		(property "LCSC" " C15401"
 			(at 934.72 290.83 90)
 			(hide yes)
@@
 			)
 		)
-		(property "Value" "SW_Push"
+		(property "Value" "TS-1101-C-W"
 			(at 81.28 608.33 0)
 			(show_name no)
@@
 			)
 		)
-		(property "Footprint" "Button_Switch_SMD:SW_SPST_EVQP2_ShortPushTravel_H2.5mm"
+		(property "Footprint" "Button_Switch_SMD:SW_Tactile_SPST_NO_Straight_CK_PTS636Sx25SMTRLFS"
 			(at 81.28 608.33 0)
 			(hide yes)
@@
 			)
 		)
+		(property "LCSC" "C318938"
+			(at 81.28 613.41 0)
+			(hide yes)
+			(show_name no)
+			(do_not_autoplace no)
+			(effects
+				(font
+					(size 1.27 1.27)
+				)
+			)
+		)
 		(pin "2"
 		)
@@
 			)
 		)
-		(property "LCSC" "C25804"
+		(property "LCSC" " C15401"
 			(at 934.72 283.21 90)
 			(hide yes)
@@
 			)
 		)
-		(property "Value" "W25Q16JVSS"
+		(property "Value" "P25Q16SH-SSH-IR"
 			(at 144.78 622.2999 0)
 			(show_name no)
@@
 			)
 		)
-		(property "LCSC" "C82317"
+		(property "LCSC" "C7466814"
 			(at 133.35 621.03 0)
 			(hide yes)
@@
 			)
 		)
-		(property "LCSC" "C25804"
+		(property "LCSC" " C15401"
 			(at 934.72 288.29 90)
 			(hide yes)
@@
 			)
 		)
-		(property "Value" "USB_C_Receptacle_USB2.0_16P"
+		(property "Value" "UC09-0B16F00P11"
 			(at 67.31 548.64 0)
 			(show_name no)
@@
 			)
 		)
-		(property "LCSC" "C3197885"
+		(property "LCSC" "C36936538"
 			(at 67.31 568.96 0)
 			(hide yes)
@@
 			)
 		)
-		(property "LCSC" "C25804"
+		(property "LCSC" " C15401"
 			(at 934.72 285.75 90)
 			(hide yes)
@@
 			)
 		)
-		(property "Value" "693063020911"
+		(property "Value" "SD-CARD 11P"
 			(at 801.37 436.88 0)
 			(hide yes)
@@
 			)
 		)
-		(property "LCSC" "C266602"
+		(property "LCSC" "C7529393"
 			(at 801.37 436.88 0)
 			(hide yes)
@@
 			)
 		)
-		(property "LCSC" "C25804"
+		(property "LCSC" " C15401"
 			(at 654.05 69.85 90)
 			(hide yes)
@@
 			)
 		)
-		(property "Value" "SW_Push"
+		(property "Value" "TS-1101-C-W"
 			(at 600.71 31.75 0)
 			(show_name no)
@@
 			)
 		)
-		(property "Footprint" "Button_Switch_SMD:SW_SPST_EVQP2_ShortPushTravel_H2.5mm"
+		(property "Footprint" "Button_Switch_SMD:SW_Tactile_SPST_NO_Straight_CK_PTS636Sx25SMTRLFS"
 			(at 600.71 31.75 0)
 			(hide yes)
@@
 			(at 600.71 36.83 0)
 			(hide yes)
+			(show_name no)
+			(do_not_autoplace no)
+			(effects
+				(font
+					(size 1.27 1.27)
+				)
+			)
+		)
+		(property "LCSC" "C318938"
+			(at 600.71 36.83 0)
+			(hide yes)

Commit message: Board cleanup
Parts:
- added TP13, TP14: TestPoint, TestPoint:TestPoint_Pad_D1.0mm, symbol Connector:TestPoint
Connections:
- net at U9.34 (GPIO22): now also TP13.1
- net at U9.37 (GPIO25): now also TP14.1
