File: v12/board/usbcart/usbcart.kicad_pcb (KiCad board)
At the start: 2 copper layers, 33 parts, among them U5 LD1117S33CTR, U81 EPM3064_44, U82 FT245RL, X1 USB-MB-S, X2 CONN_02X05, X3 CONN_02X05, X4 CONN_01X01

Commit message: Minor changes to boards
- Added chip orientation information for 3V3 buffers and MAX10
footprints
- Added gerber files
Other:
- board text added: "Mfg. date : 2016 July 14"
- board text removed: "Mfg. date : 2016 July 11"
Changed lines of the file:
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@@
   (title_block
     (title "USB Mezzanine Board")
-    (date 2016-07-09)
+    (date 2016-07-14)
     (rev 4.1)
-    (company cafe-alpha)
+    (company "cafe-alpha (http://ppcenter.free.fr/satcart/)")
     (comment 2 "Distributed under GNU GENERAL PUBLIC LICENSE Version 2")
   )
@@
       (xy -10.49782 1.94818) (xy 10.33018 1.94818) (xy 10.33018 -2.032) (xy 10.33018 -2.032)) (layer B.SilkS) (width 0.00254))
   )
-  (gr_text "Mfg. date :\n2016 July 11" (at 102.1 127.4) (layer F.SilkS)
+  (gr_text "Mfg. date :\n2016 July 14" (at 102.1 127.4) (layer F.SilkS)
     (effects (font (size 0.8992 0.8992) (thickness 0.1905)))
   )
