File: v12/board/wasca/wasca.kicad_pcb (KiCad board)
At the start: 2 copper layers, 74 parts, among them CN1 CARTRIDGE_EDGE_CONNECTOR, P84 CONN_01X02, U1 74ALVC164245, U11 74ALVC164245, U2 74ALVC164245, U3 74ALVC164245, U4 74ALVC164245, U5 LD1117S33CTR, U8 10M08SCE144I7G, U9 SDRAM_MT48_x16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

Commit message: Minor changes to boards
- Added chip orientation information for 3V3 buffers and MAX10
footprints
- Added gerber files
Parts:
- U1, U11, U2, U3, U4: footprint Housings_SSOP:TSSOP-48_6.1x12.5mm_Pitch0.5mm -> wasca:TSSOP-48_6.1x12.5mm_Pitch0.5mm
Other:
- board text added: "Mfg. date : 2016 July 14"
- board text removed: "Mfg. date : 2016 July 11"
